File: hardware/kicad/bwlr3d.kicad_sch (KiCad schematic)
At the start: 103 parts, among them Q1 AO3407, Q2 DMG1012UW, Q3 PMV32UP, Q4 DMG1012UW, SW3 RESET, SW4 BOOT, U1 BME680, U2 RAK3172, U3 AEM10941-QFN, U4 XC6215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

Commit message: update library and footprint
Changed lines of the file:
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@@
   (symbol (lib_name "Solar_Cell_1") (lib_id "Device:Solar_Cell") (at 21.59 25.4 0) (unit 1)
     (in_bom yes) (on_board yes)
-    (property "Reference" "SC3" (id 0) (at 25.4 21.9709 0)
-      (effects (font (size 1.27 1.27)) (justify left))
-    )
-    (property "Value" "KXOB25-05X3F" (id 1) (at 17.78 16.51 0)
+    (property "Reference" "SC3" (id 0) (at 24.13 23.114 0)
+      (effects (font (size 1.27 1.27)) (justify left))
+    )
+    (property "Value" "KXOB25-05X3F" (id 1) (at 23.876 25.654 0)
       (effects (font (size 1.27 1.27)) (justify left))
     )
@@
   (symbol (lib_name "Solar_Cell_1") (lib_id "Device:Solar_Cell") (at 21.59 47.625 0) (unit 1)
     (in_bom yes) (on_board yes)
-    (property "Reference" "SC4" (id 0) (at 25.4 44.1959 0)
-      (effects (font (size 1.27 1.27)) (justify left))
-    )
-    (property "Value" "KXOB25-05X3F" (id 1) (at 13.97 38.735 0)
-      (effects (font (size 1.27 1.27)) (justify left))
-    )
+    (property "Reference" "SC4" (id 0) (at 24.384 44.958 0)
+      (effects (font (size 1.27 1.27)) (justify left))
+    )
+    (property "Value" "KXOB25-05X3F" (id 1) (at 24.003 47.498 0)
+      (effects (font (size 1.27 1.27)) (justify left))
+    )

Commit message: switch IMU_INT with BATT_MEAS, switch I2C pull-up to 3V3P, and add GND stitch
Connections:
- net +3.3V: no longer R6.1, R7.1
- net +3.3VP: now also R6.1, R7.1
- net BATT_MEAS: now also U2.31 (PB4/ADC2); no longer U2.25 (PA10/ADC4)
- net IMU_INT: now also U2.25 (PA10/ADC4); no longer U2.31 (PB4/ADC2)
Changed lines of the file:
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@@
     (stroke (width 0) (type default) (color 0 0 0 0))
   )
-  (wire (pts (xy 60.325 143.51) (xy 71.755 143.51))
-    (stroke (width 0) (type default) (color 0 0 0 0))
-  )
   (wire (pts (xy 88.265 214.63) (xy 104.14 214.63))
     (stroke (width 0) (type default) (color 0 0 0 0))
@@
     (stroke (width 0) (type default) (color 0 0 0 0))
   )
+  (wire (pts (xy 61.214 138.43) (xy 71.755 138.43))
+    (stroke (width 0) (type default) (color 0 0 0 0))
+  )
   (wire (pts (xy 98.425 168.91) (xy 98.425 170.18))
     (stroke (width 0) (type default) (color 0 0 0 0))
@@
     (stroke (width 0) (type default) (color 0 0 0 0))
   )
-  (wire (pts (xy 64.135 138.43) (xy 71.755 138.43))
-    (stroke (width 0) (type default) (color 0 0 0 0))
-  )
   (wire (pts (xy 95.25 21.59) (xy 85.09 21.59))
     (stroke (width 0) (type default) (color 0 0 0 0))
@@
     (stroke (width 0) (type default) (color 0 0 0 0))
   )
+  (wire (pts (xy 63.881 143.51) (xy 71.755 143.51))
+    (stroke (width 0) (type default) (color 0 0 0 0))
+  )
   (wire (pts (xy 368.935 140.97) (xy 368.935 146.05))
     (stroke (width 0) (type default) (color 0 0 0 0))
@@
     (effects (font (size 1.27 1.27)) (justify right bottom))
   )
-  (label "BATT_MEAS" (at 60.325 143.51 0)
+  (label "BATT_MEAS" (at 61.214 138.43 0)
     (effects (font (size 1.27 1.27)) (justify left bottom))
   )
@@
     (effects (font (size 1.27 1.27)) (justify left bottom))
   )
-  (label "IMU_INT" (at 64.135 138.43 0)
+  (label "IMU_INT" (at 63.881 143.51 0)
     (effects (font (size 1.27 1.27)) (justify left bottom))
   )
@@
     (pin "2")
   )
-  (symbol (lib_id "power:+3.3V") (at 142.875 118.11 0) (mirror y) (unit 1)
-    (in_bom yes) (on_board yes)
-    (property "Reference" "#PWR0119" (id 0) (at 142.875 121.92 0)
-      (effects (font (size 1.27 1.27)) hide)
-    )
-    (property "Value" "+3.3V" (id 1) (at 147.955 116.205 0))
-    (property "Footprint" "" (id 2) (at 142.875 118.11 0)
-      (effects (font (size 1.27 1.27)) hide)
-    )
-    (property "Datasheet" "" (id 3) (at 142.875 118.11 0)
-      (effects (font (size 1.27 1.27)) hide)
-    )
-    (pin "1")
-  )
   (symbol (lib_id "power:GND") (at 156.21 60.96 0) (unit 1)
     (in_bom yes) (on_board yes)
@@
     (pin "1")
   )
-  (symbol (lib_id "power:+3.3V") (at 135.255 118.11 0) (unit 1)
-    (in_bom yes) (on_board yes)
-    (property "Reference" "#PWR0114" (id 0) (at 135.255 121.92 0)
-      (effects (font (size 1.27 1.27)) hide)
-    )
-    (property "Value" "+3.3V" (id 1) (at 130.175 116.205 0))
-    (property "Footprint" "" (id 2) (at 135.255 118.11 0)
-      (effects (font (size 1.27 1.27)) hide)
-    )
-    (property "Datasheet" "" (id 3) (at 135.255 118.11 0)
-      (effects (font (size 1.27 1.27)) hide)
-    )
-    (pin "1")
-  )
   (symbol (lib_id "Jumper:SolderJumper_3_Open") (at 285.75 37.465 270) (unit 1)
     (in_bom yes) (on_board yes)
@@
     (pin "1")
   )
+  (symbol (lib_id "power:+3.3VP") (at 135.255 118.11 0) (unit 1)
+    (in_bom yes) (on_board yes)
+    (property "Reference" "#PWR0119" (id 0) (at 139.065 119.38 0)
+      (effects (font (size 1.27 1.27)) hide)
+    )
+    (property "Value" "+3.3VP" (id 1) (at 134.62 114.3 0))
+    (property "Footprint" "" (id 2) (at 135.255 118.11 0)
+      (effects (font (size 1.27 1.27)) hide)
+    )
+    (property "Datasheet" "" (id 3) (at 135.255 118.11 0)
+      (effects (font (size 1.27 1.27)) hide)
+    )
+    (pin "1")
+  )
   (symbol (lib_id "Switch:SW_Push") (at 40.005 130.81 90) (unit 1)
     (in_bom yes) (on_board yes)
@@
     (pin "2")
   )
+  (symbol (lib_id "power:+3.3VP") (at 142.875 118.11 0) (unit 1)
+    (in_bom yes) (on_board yes)
+    (property "Reference" "#PWR0114" (id 0) (at 146.685 119.38 0)
+      (effects (font (size 1.27 1.27)) hide)
+    )
+    (property "Value" "+3.3VP" (id 1) (at 143.51 114.3 0))
+    (property "Footprint" "" (id 2) (at 142.875 118.11 0)
+      (effects (font (size 1.27 1.27)) hide)
+    )
+    (property "Datasheet" "" (id 3) (at 142.875 118.11 0)
+      (effects (font (size 1.27 1.27)) hide)
+    )
+    (pin "1")
+  )
   (symbol (lib_id "power:GND") (at 250.19 240.665 0) (unit 1)
     (in_bom yes) (on_board yes)
@@
       (reference "#PWR0113") (unit 1) (value "GND") (footprint "")
     )
-    (path "/709c1fbd-24ac-4a6e-91dd-33444481cc8f"
-      (reference "#PWR0114") (unit 1) (value "+3.3V") (footprint "")
+    (path "/f5dbfdd3-affe-43c2-ba80-a1e95c85b91a"
+      (reference "#PWR0114") (unit 1) (value "+3.3VP") (footprint "")
     )
     (path "/baf8d7be-2723-4be7-a268-2213f3fd7183"
@@
       (reference "#PWR0118") (unit 1) (value "GND") (footprint "")
     )
-    (path "/43ebd406-e344-4ae6-a57a-c8a9c0e0361e"
-      (reference "#PWR0119") (unit 1) (value "+3.3V") (footprint "")
+    (path "/7cb82e06-f3de-4747-9506-8f54668ce182"
+      (reference "#PWR0119") (unit 1) (value "+3.3VP") (footprint "")
     )
     (path "/7ee2cb5d-cd26-44e1-8e2b-a9fa6d535684"

Commit message: change voltage divider value to 4.7K and 10K, add 0.1uF capacitor to voltage divider
Parts:
- added C35: 0.1uF, Capacitor_SMD:C_0603_1608Metric, symbol Device:C
- R1: value 4.7M -> 4.7K
- R4: value 10M -> 10K
Connections:
- net BATT_MEAS: now also C35.2
- net GND: now also C35.1
Changed lines of the file:
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@@
   (junction (at 90.805 83.82) (diameter 0) (color 0 0 0 0)
   )
+  (junction (at 264.16 168.91) (diameter 0) (color 0 0 0 0)
+  )
   (junction (at 396.875 71.755) (diameter 0) (color 0 0 0 0)
   )
+  (junction (at 273.05 180.34) (diameter 0) (color 0 0 0 0)
+  )
   (junction (at 278.765 37.465) (diameter 0) (color 0 0 0 0)
   )
@@
     (stroke (width 0) (type default) (color 0 0 0 0))
   )
+  (wire (pts (xy 264.16 168.91) (xy 264.16 171.45))
+    (stroke (width 0) (type default) (color 0 0 0 0))
+  )
   (wire (pts (xy 32.385 179.07) (xy 32.385 181.61))
     (stroke (width 0) (type default) (color 0 0 0 0))
@@
     (stroke (width 0) (type default) (color 0 0 0 0))
   )
+  (wire (pts (xy 264.16 180.34) (xy 273.05 180.34))
+    (stroke (width 0) (type default) (color 0 0 0 0))
+  )
   (wire (pts (xy 45.72 207.01) (xy 42.545 207.01))
     (stroke (width 0) (type default) (color 0 0 0 0))
@@
     (stroke (width 0) (type default) (color 0 0 0 0))
   )
+  (wire (pts (xy 264.16 168.91) (xy 273.05 168.91))
+    (stroke (width 0) (type default) (color 0 0 0 0))
+  )
   (polyline (pts (xy 238.76 193.675) (xy 325.755 193.675))
     (stroke (width 0) (type default) (color 0 0 0 0))
@@
     (stroke (width 0) (type default) (color 0 0 0 0))
   )
+  (wire (pts (xy 252.73 168.91) (xy 264.16 168.91))
+    (stroke (width 0) (type default) (color 0 0 0 0))
+  )
   (wire (pts (xy 95.885 168.91) (xy 95.885 170.18))
     (stroke (width 0) (type default) (color 0 0 0 0))
@@
     (stroke (width 0) (type default) (color 0 0 0 0))
   )
-  (wire (pts (xy 273.05 177.165) (xy 273.05 180.975))
+  (wire (pts (xy 273.05 177.165) (xy 273.05 180.34))
     (stroke (width 0) (type default) (color 0 0 0 0))
   )
@@
     (stroke (width 0) (type default) (color 0 0 0 0))
   )
-  (wire (pts (xy 259.08 168.91) (xy 273.05 168.91))
-    (stroke (width 0) (type default) (color 0 0 0 0))
-  )
   (wire (pts (xy 273.05 140.97) (xy 273.05 142.875))
     (stroke (width 0) (type default) (color 0 0 0 0))
@@
     (stroke (width 0) (type default) (color 0 0 0 0))
   )
+  (wire (pts (xy 264.16 179.07) (xy 264.16 180.34))
+    (stroke (width 0) (type default) (color 0 0 0 0))
+  )
   (wire (pts (xy 278.765 37.465) (xy 281.94 37.465))
     (stroke (width 0) (type default) (color 0 0 0 0))
@@
     (stroke (width 0) (type default) (color 0 0 0 0))
   )
+  (wire (pts (xy 273.05 180.34) (xy 273.05 180.975))
+    (stroke (width 0) (type default) (color 0 0 0 0))
+  )
   (wire (pts (xy 52.705 123.19) (xy 52.705 128.27))
     (stroke (width 0) (type default) (color 0 0 0 0))
@@
     (effects (font (size 1.27 1.27)) (justify right bottom))
   )
-  (label "BATT_MEAS" (at 259.08 168.91 0)
+  (label "BATT_MEAS" (at 252.73 168.91 0)
     (effects (font (size 1.27 1.27)) (justify left bottom))
   )
@@
       (effects (font (size 1.27 1.27)) (justify left))
     )
-    (property "Value" "4.7M" (id 1) (at 275.59 165.7349 0)
+    (property "Value" "4.7K" (id 1) (at 275.59 165.7349 0)
       (effects (font (size 1.27 1.27)) (justify left))
     )
@@
     (pin "2")
   )
+  (symbol (lib_id "Device:C") (at 264.16 175.26 180) (unit 1)
+    (in_bom yes) (on_board yes)
+    (property "Reference" "C35" (id 0) (at 262.255 172.72 0)
+      (effects (font (size 1.27 1.27)) (justify left))
+    )
+    (property "Value" "0.1uF" (id 1) (at 263.525 177.8 0)
+      (effects (font (size 1.27 1.27)) (justify left))
+    )
+    (property "Footprint" "Capacitor_SMD:C_0603_1608Metric" (id 2) (at 263.1948 171.45 0)
+      (effects (font (size 1.27 1.27)) hide)
+    )
+    (property "Datasheet" "~" (id 3) (at 264.16 175.26 0)
+      (effects (font (size 1.27 1.27)) hide)
+    )
+    (pin "1")
+    (pin "2")
+  )
   (symbol (lib_id "power:GND") (at 45.085 181.61 0) (unit 1)
     (in_bom yes) (on_board yes)
@@
       (effects (font (size 1.27 1.27)) (justify left))
     )
-    (property "Value" "10M" (id 1) (at 275.59 175.8949 0)
+    (property "Value" "10K" (id 1) (at 275.59 175.8949 0)
       (effects (font (size 1.27 1.27)) (justify left))
     )
@@
       (reference "C34") (unit 1) (value "10uF") (footprint "Capacitor_SMD:C_0603_1608Metric")
     )
+    (path "/a775b801-772d-4ebc-8ef8-95b9697f26de"
+      (reference "C35") (unit 1) (value "0.1uF") (footprint "Capacitor_SMD:C_0603_1608Metric")
+    )
     (path "/c843fb3d-2518-420f-851e-a463adcfffc8"
       (reference "D1") (unit 1) (value "RED") (footprint "LED_SMD:LED_0603_1608Metric")
@@
     )
     (path "/a5b89eaf-e950-409e-8cf0-5337008b2aea"
-      (reference "R1") (unit 1) (value "4.7M") (footprint "Resistor_SMD:R_0603_1608Metric")
+      (reference "R1") (unit 1) (value "4.7K") (footprint "Resistor_SMD:R_0603_1608Metric")
     )
     (path "/d1598165-620d-4060-bc1e-5d119f5ebb8f"
@@
     )
     (path "/e77c86b9-325a-4d07-b085-8c7758806002"
-      (reference "R4") (unit 1) (value "10M") (footprint "Resistor_SMD:R_0603_1608Metric")
+      (reference "R4") (unit 1) (value "10K") (footprint "Resistor_SMD:R_0603_1608Metric")
     )
     (path "/93436335-fd4e-48d0-8d58-12ac441e8361"

Commit message: release board revision 1
Other:
- company: (none) -> Teapot Laboratories
- title: (none) -> Teapot BWLR3D
Changed lines of the file:
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@@
 (kicad_sch (version 20211123) (generator eeschema)
   (paper "A3")
+  (title_block
+    (title "Teapot BWLR3D")
+    (date "2022-11-08")
+    (rev "1")
+    (company "Teapot Laboratories")
+  )
   (junction (at 176.53 60.96) (diameter 0) (color 0 0 0 0)
   )
